Commit message: added readme

File: proxygen_description/xacro/proxygen.xacro (robot description, xacro)
@@ -3,5 +3,5 @@
 <robot xmlns:xacro="http://ros.org/wiki/xacro">
 <xacro:property name="base_radii" value="0.100"/>
-<!-- height from the ground to the base plate -->
+<!-- height from the ground to the top of the base plate -->
 <xacro:property name="base_height" value="0.180"/>
 <xacro:property name="base_plate_thickness" value="0.010"/>
@@ -173,5 +173,5 @@
       <origin xyz="0 0 0" rpy="0 0 0"/>
       <geometry>
-        <mesh filename="package://proxygen_description/meshes/chain_link5.stl" scale="0.001 0.001 0.001"/>
+        <mesh filename="$(find proxygen_description)/meshes/chain_link5.stl" scale="0.001 0.001 0.001"/>
       </geometry>
       <material name="grey"/>
@@ -180,5 +180,5 @@
       <origin xyz="0 0 0" rpy="0 0 0"/>
       <geometry>
-        <mesh filename="package://proxygen_description/meshes/chain_link5.stl" scale="0.001 0.001 0.001"/>
+        <mesh filename="$(find proxygen_description)/meshes/chain_link5.stl" scale="0.001 0.001 0.001"/>
       </geometry>
     </collision>
@@ -196,5 +196,5 @@
       <origin xyz="0.0 0.0 0" rpy="0 0 0"/>
       <geometry>
-        <mesh filename="package://proxygen_description/meshes/chain_link_grip_l.stl" scale="0.001 0.001 0.001"/>
+        <mesh filename="$(find proxygen_description)/meshes/chain_link_grip_l.stl" scale="0.001 0.001 0.001"/>
       </geometry>
       <material name="grey"/>
@@ -203,5 +203,5 @@
       <origin xyz="0.0 0.0 0" rpy="0 0 0"/>
       <geometry>
-        <mesh filename="package://proxygen_description/meshes/chain_link_grip_l.stl" scale="0.001 0.001 0.001"/>
+        <mesh filename="$(find proxygen_description)/meshes/chain_link_grip_l.stl" scale="0.001 0.001 0.001"/>
       </geometry>
     </collision>
@@ -227,5 +227,5 @@
       <origin xyz="0.0 -0.0 0" rpy="0 0 0"/>
       <geometry>
-        <mesh filename="package://proxygen_description/meshes/chain_link_grip_r.stl" scale="0.001 0.001 0.001"/>
+        <mesh filename="$(find proxygen_description)/meshes/chain_link_grip_r.stl" scale="0.001 0.001 0.001"/>
       </geometry>
       <material name="grey"/>
@@ -234,5 +234,5 @@
       <origin xyz="0.0 -0.0 0" rpy="0 0 0"/>
       <geometry>
-        <mesh filename="package://proxygen_description/meshes/chain_link_grip_r.stl" scale="0.001 0.001 0.001"/>
+        <mesh filename="$(find proxygen_description)/meshes/chain_link_grip_r.stl" scale="0.001 0.001 0.001"/>
       </geometry>
     </collision>

Commit message: launch file for gazebo, donegit status

File: proxygen_description/xacro/proxygen.xacro (robot description, xacro)
@@ -102,6 +102,5 @@
     <origin xyz="0.0 0.0 0.060" rpy="0 0 0"/>
     <axis xyz="0 1 0"/>
-    <!-- <limit velocity="4.8" effort="1" lower="${-pi*0.57}" upper="${pi*0.5}" /> -->
-    <limit velocity="4.8" effort="1" lower="${-1.0}" upper="${1.3}" />
+    <limit velocity="4.8" effort="1" lower="${-pi * 0.9 / 2}" upper="${pi * 0.9 / 2}" />
   </joint>
   <xacro:Supp_Link parent="arm1" x="0" y="0" z="0.0" height="0.060"/>
@@ -122,5 +121,5 @@
     </collision>
     <inertial>
-      <origin xyz="1.0308393e-02 3.7743363e-04 1.0170197e-01" />
+      <origin xyz="0 0 ${arm1_length/2}" />
       <mass value="1.3850917e-01" />
       <inertia ixx="3.3055381e-04" ixy="-9.7940978e-08" ixz="-3.8505711e-05"
@@ -135,6 +134,5 @@
     <origin xyz="0.0 0.045 ${arm2_joint_height}" rpy="0 1.57 0"/>
     <axis xyz="0 1 0"/>
-    <limit velocity="4.8" effort="1" lower="${-pi / 2 * 0.8}" upper="${pi / 2 * 0.8}" />
-    <!-- <limit velocity="4.8" effort="1" lower="${-pi}" upper="${pi}" /> -->
+    <limit velocity="4.8" effort="1" lower="${-pi * 0.8 / 2}" upper="${pi * 0.8 / 2}" />
   </joint>
   <xacro:Supp_Link parent="arm2" x="0" y="-0.025" z="0" height="0.100"/>
@@ -155,5 +153,5 @@
     </collision>
     <inertial>
-      <origin xyz="9.0909590e-02 3.8929816e-04 2.2413279e-04" />
+      <origin xyz="0 0 ${arm2_length/2}" />
       <mass value="1.3274562e-01" />
       <inertia ixx="3.0654178e-05" ixy="-1.2764155e-06" ixz="-2.6874417e-07"

Commit message: solved: stl files weren't loading in rviz: syntax issue

File: proxygen_description/xacro/proxygen.xacro (robot description, xacro)
@@ -171,5 +171,5 @@
       <origin xyz="0 0 0" rpy="0 0 0"/>
       <geometry>
-        <mesh filename="$(find proxygen_description)/meshes/chain_link5.stl" scale="0.001 0.001 0.001"/>
+        <mesh filename="file://$(find proxygen_description)/meshes/chain_link5.stl" scale="0.001 0.001 0.001"/>
       </geometry>
       <material name="grey"/>
@@ -178,5 +178,5 @@
       <origin xyz="0 0 0" rpy="0 0 0"/>
       <geometry>
-        <mesh filename="$(find proxygen_description)/meshes/chain_link5.stl" scale="0.001 0.001 0.001"/>
+        <mesh filename="file://$(find proxygen_description)/meshes/chain_link5.stl" scale="0.001 0.001 0.001"/>
       </geometry>
     </collision>
@@ -194,5 +194,5 @@
       <origin xyz="0.0 0.0 0" rpy="0 0 0"/>
       <geometry>
-        <mesh filename="$(find proxygen_description)/meshes/chain_link_grip_l.stl" scale="0.001 0.001 0.001"/>
+        <mesh filename="file://$(find proxygen_description)/meshes/chain_link_grip_l.stl" scale="0.001 0.001 0.001"/>
       </geometry>
       <material name="grey"/>
@@ -201,5 +201,5 @@
       <origin xyz="0.0 0.0 0" rpy="0 0 0"/>
       <geometry>
-        <mesh filename="$(find proxygen_description)/meshes/chain_link_grip_l.stl" scale="0.001 0.001 0.001"/>
+        <mesh filename="file://$(find proxygen_description)/meshes/chain_link_grip_l.stl" scale="0.001 0.001 0.001"/>
       </geometry>
     </collision>
@@ -225,5 +225,5 @@
       <origin xyz="0.0 -0.0 0" rpy="0 0 0"/>
       <geometry>
-        <mesh filename="$(find proxygen_description)/meshes/chain_link_grip_r.stl" scale="0.001 0.001 0.001"/>
+        <mesh filename="file://$(find proxygen_description)/meshes/chain_link_grip_r.stl" scale="0.001 0.001 0.001"/>
       </geometry>
       <material name="grey"/>
@@ -232,5 +232,5 @@
       <origin xyz="0.0 -0.0 0" rpy="0 0 0"/>
       <geometry>
-        <mesh filename="$(find proxygen_description)/meshes/chain_link_grip_r.stl" scale="0.001 0.001 0.001"/>
+        <mesh filename="file://$(find proxygen_description)/meshes/chain_link_grip_r.stl" scale="0.001 0.001 0.001"/>
       </geometry>
     </collision>
