Commit message: added rotation axis (dummy link)

File: proxygen_description/xacro/proxygen.full.xacro (robot description, xacro)
@@ -2,20 +2,4 @@
 <!-- Open_Manipulator Chain -->
 <robot name="proxygen" xmlns:xacro="http://ros.org/wiki/xacro">
-    <xacro:property name="base_radii" value="0.100"/>
-    <!-- height from the ground to the base plate -->
-    <xacro:property name="base_height" value="0.180"/>
-    <xacro:property name="base_plate_thickness" value="0.010"/>
-    <xacro:property name="base_plate_radii" value="0.070"/>
-    <xacro:property name="base_plate_distance" value="0.010"/>
-    <!-- arm1 joint height from the base plate -->
-    <xacro:property name="arm1_joint_height" value="0.060"/>
-    <xacro:property name="arm1_width" value="0.040"/>
-    <!-- arm2 joint height from the joint1 -->
-    <xacro:property name="arm2_joint_height" value="0.400"/>
-    <xacro:property name="arm2_width" value="0.040"/>
-    <xacro:property name="end_effector_joint_height" value="0.350"/>
-    <xacro:property name="end_effector_joint_offset" value="0.050"/>
-    <xacro:property name="arm1_length" value="${arm2_joint_height - arm1_width * 1.5 / 2}"/>
-    <xacro:property name="arm2_length" value="${end_effector_joint_height - end_effector_joint_offset}"/>
     <material name="black">
         <color rgba="0.0 0.0 0.0 1.0"/>
@@ -30,27 +14,4 @@
         <color rgba="0.5 0.5 0.5 1.0"/>
     </material>
-    <xacro:macro name="Supp_Link" params="parent x y z height">
-        <link name="supp_link${parent}">
-        <visual>
-            <origin xyz="0 0 0" rpy="-1.57 0 0"/>
-            <geometry>
-            <cylinder radius="0.04" length="${height}"/>
-            </geometry>
-            <material name="blue"/>
-        </visual>
-        <inertial>
-            <origin xyz="0 0 0" />
-            <mass value="9.8406837e-03" />
-            <inertia ixx="3.4543422e-06" ixy="-1.6031095e-07" ixz="-3.8375155e-08"
-                    iyy="3.2689329e-06"  iyz="2.8511935e-07"
-                    izz="1.8850320e-06" />
-        </inertial>
-        </link>
-        <joint name="supp_joint${parent}" type="fixed">
-        <parent link="${parent}"/>
-        <child link="supp_link${parent}"/>
-        <origin xyz="${x} ${y} ${z}" rpy="0 0 0"/>
-        </joint>
-    </xacro:macro>
     <!-- World -->
     <link name="world"/>
@@ -67,125 +28,178 @@
         <child link="base_link"/>
     </joint>
-    <!-- Base_Link -->
-    <link name="base_link">
-        <visual>
-        <origin xyz="0.0 0.0 ${base_height/2 - base_plate_thickness/2 - base_plate_distance/2}" rpy="0 0 0"/>
+<xacro:property name="base_radii" value="0.100"/>
+<!-- height from the ground to the top of the base plate -->
+<xacro:property name="base_height" value="0.180"/>
+<xacro:property name="base_plate_thickness" value="0.010"/>
+<xacro:property name="base_plate_radii" value="0.070"/>
+<xacro:property name="base_plate_distance" value="0.010"/>
+<!-- arm1 joint height from the base plate -->
+<xacro:property name="arm1_joint_height" value="0.060"/>
+<xacro:property name="arm1_width" value="0.040"/>
+<!-- arm2 joint height from the joint1 -->
+<xacro:property name="arm2_joint_height" value="0.400"/>
+<xacro:property name="arm2_width" value="0.040"/>
+<xacro:property name="end_effector_joint_height" value="0.350"/>
+<xacro:property name="end_effector_joint_offset" value="0.050"/>
+<xacro:property name="arm1_length" value="${arm2_joint_height - arm1_width * 1.5 / 2}"/>
+<xacro:property name="arm2_length" value="${end_effector_joint_height}"/>
+  <xacro:macro name="Supp_Link" params="parent x y z height">
+    <link name="supp_link${parent}">
+      <visual>
+        <origin xyz="0 0 0" rpy="-1.57 0 0"/>
         <geometry>
-            <cylinder radius="${base_radii}" length="${base_height - base_plate_thickness - base_plate_distance}"/>
+          <cylinder radius="0.04" length="${height}"/>
         </geometry>
-        <material name="grey"/>
-        </visual>
-        <collision>
-        <origin xyz="0.0 0.0 ${base_height/2 - base_plate_thickness/2 - base_plate_distance/2}" rpy="0 0 0"/>
-        <geometry>
-            <cylinder radius="${base_radii}" length="${base_height - base_plate_thickness - base_plate_distance}"/>
-        </geometry>
-        </collision>
-        <inertial>
-        <origin xyz="3.0876154e-04 0.0000000e+00 -1.2176461e-04" />
-        <mass value="7.9119962e-02" />
-        <inertia ixx="1.2505234e-05" ixy="0.0" ixz="-1.7855208e-07"
-                iyy="2.1898364e-05" iyz="0.0"
-                izz="1.9267361e-05" />
-        </inertial>
+        <material name="blue"/>
+      </visual>
+      <inertial>
+        <origin xyz="0 0 0" />
+        <mass value="9.8406837e-03" />
+        <inertia ixx="3.4543422e-06" ixy="-1.6031095e-07" ixz="-3.8375155e-08"
+                 iyy="3.2689329e-06"  iyz="2.8511935e-07"
+                 izz="1.8850320e-06" />
+      </inertial>
     </link>
-    <!-- Base_Link_Plate_Joint -->
-    <joint name="base_link_plate_joint" type="revolute">
-        <parent link="base_link"/>
-        <child link="base_plate"/>
-        <origin xyz="0.0 0.0 ${base_height}" rpy="0 0 0"/>
-        <axis xyz="0 0 1"/>
-        <limit velocity="4.8" effort="1" lower="${-pi*0.9}" upper="${pi*0.9}"/>
-        <!-- <limit velocity="4.8" effort="1" lower="${-pi/2}" upper="${pi/2}" /> -->
+    <joint name="supp_joint${parent}" type="fixed">
+      <parent link="${parent}"/>
+      <child link="supp_link${parent}"/>
+      <origin xyz="${x} ${y} ${z}" rpy="0 0 0"/>
     </joint>
-    <!--  Base_Plate -->
-    <link name="base_plate">
-        <visual>
-        <origin xyz="0 0 ${-base_plate_thickness/2}" rpy="0 0 0"/>
-        <geometry>
-            <cylinder radius="${base_plate_radii}" length="${base_plate_thickness}"/>
-        </geometry>
-        <material name="black"/>
-        </visual>
-        <collision>
-        <origin xyz="0 0 ${-base_plate_thickness/2}" rpy="0 0 0"/>
-        <geometry>
-            <cylinder radius="${base_plate_radii}" length="${base_plate_thickness}"/>
-        </geometry>
-        </collision>
-        <inertial>
-        <origin xyz="-3.0184870e-04 5.4043684e-04 ${0.018 + 2.9433464e-02}" />
-        <mass value="9.8406837e-02" />
-        <inertia ixx="3.4543422e-05" ixy="-1.6031095e-08" ixz="-3.8375155e-07"
-                iyy="3.2689329e-05" iyz="2.8511935e-08"
-                izz="1.8850320e-05" />
-        </inertial>
-    </link>
-    <!--  Base_Plate_Arm1_Joint -->
-    <joint name="base_plate_arm1_joint" type="revolute">
-        <parent link="base_plate"/>
-        <child link="arm1"/>
-        <origin xyz="0.0 0.0 0.060" rpy="0 0 0"/>
-        <axis xyz="0 1 0"/>
-        <!-- <limit velocity="4.8" effort="1" lower="${-pi*0.57}" upper="${pi*0.5}" /> -->
-        <limit velocity="4.8" effort="1" lower="${-1.0}" upper="${1.3}" />
-    </joint>
-    <xacro:Supp_Link parent="arm1" x="0" y="0" z="0.0" height="0.060"/>
-    <!--  Arm1 -->
-    <link name="arm1">
-        <visual>
-        <origin xyz="0 0 ${arm1_length/2}" rpy="0 0 0"/>
-        <geometry>
-            <box size="${arm1_width} ${arm1_width} ${arm1_length}"/>
-        </geometry>
-        <material name="black"/>
-        </visual>
-        <collision>
-        <origin xyz="0 0 ${arm1_length/2}" rpy="0 0 0"/>
-        <geometry>
-            <box size="${arm1_width} ${arm1_width} ${arm1_length}"/>
-        </geometry>
-        </collision>
-        <inertial>
-        <origin xyz="1.0308393e-02 3.7743363e-04 1.0170197e-01" />
-        <mass value="1.3850917e-01" />
-        <inertia ixx="3.3055381e-04" ixy="-9.7940978e-08" ixz="-3.8505711e-05"
-                iyy="3.4290447e-04" iyz="-1.5717516e-06"
-                izz="6.0346498e-05" />
-        </inertial>
-    </link>
-    <!--  Base_Plate_Arm2_Joint -->
-    <joint name="arm1_arm2_joint" type="revolute">
-        <parent link="arm1"/>
-        <child link="arm2"/>
-        <origin xyz="0.0 0.045 ${arm2_joint_height}" rpy="0 1.57 0"/>
-        <axis xyz="0 1 0"/>
-        <limit velocity="4.8" effort="1" lower="${-pi / 2 * 0.8}" upper="${pi / 2 * 0.8}" />
-        <!-- <limit velocity="4.8" effort="1" lower="${-pi}" upper="${pi}" /> -->
-    </joint>
-    <xacro:Supp_Link parent="arm2" x="0" y="-0.025" z="0" height="0.100"/>
-    <!--  Arm2 -->
-    <link name="arm2">
-        <visual>
-        <origin xyz="0 0 ${arm2_length/2}" rpy="0 0 0"/>
-        <geometry>
-            <box size="${arm2_width} ${arm2_width} ${arm2_length}"/>
-        </geometry>
-        <material name="black"/>
-        </visual>
-        <collision>
-        <origin xyz="0 0 ${arm2_length/2}" rpy="0 0 0"/>
-        <geometry>
-            <box size="${arm2_width} ${arm2_width} ${arm2_length}"/>
-        </geometry>
-        </collision>
-        <inertial>
-        <origin xyz="9.0909590e-02 3.8929816e-04 2.2413279e-04" />
-        <mass value="1.3274562e-01" />
-        <inertia ixx="3.0654178e-05" ixy="-1.2764155e-06" ixz="-2.6874417e-07"
-                iyy="2.4230292e-04" iyz="1.1559550e-08"
-                izz="2.5155057e-04" />
-        </inertial>
-    </link>
+  </xacro:macro>
+  <!-- Base_Link -->
+  <link name="base_link">
+    <visual>
+      <origin xyz="0.0 0.0 ${base_height/2 - base_plate_thickness/2 - base_plate_distance/2}" rpy="0 0 0"/>
+      <geometry>
+        <cylinder radius="${base_radii}" length="${base_height - base_plate_thickness - base_plate_distance}"/>
+      </geometry>
+      <material name="grey"/>
+    </visual>
+    <collision>
+      <origin xyz="0.0 0.0 ${base_height/2 - base_plate_thickness/2 - base_plate_distance/2}" rpy="0 0 0"/>
+      <geometry>
+        <cylinder radius="${base_radii}" length="${base_height - base_plate_thickness - base_plate_distance}"/>
+      </geometry>
+    </collision>
+    <inertial>
+      <origin xyz="3.0876154e-04 0.0000000e+00 -1.2176461e-04" />
+      <mass value="7.9119962e-02" />
+      <inertia ixx="1.2505234e-05" ixy="0.0" ixz="-1.7855208e-07"
+               iyy="2.1898364e-05" iyz="0.0"
+               izz="1.9267361e-05" />
+    </inertial>
+  </link>
+  <!-- Dummy_Link -->
+  <link name="dummy_link">
+    <visual>
+      <origin xyz="0.0 0.0 ${base_height/2 + arm1_joint_height/2}" rpy="0 0 0"/>
+      <geometry>
+        <cylinder radius="0.030" length="${base_height + arm1_joint_height}"/>
+      </geometry>
+      <material name="grey"/>
+    </visual>
+  </link>
+  <!-- Dummy_Joint -->
+  <joint name="dummy_joint" type="fixed">
+    <parent link="base_link"/>
+    <child link="dummy_link"/>
+    <origin xyz="0 0 0" rpy="0 0 0"/>
+  </joint>
+  <!-- Base_Link_Plate_Joint -->
+  <joint name="base_link_plate_joint" type="revolute">
+    <parent link="base_link"/>
+    <child link="base_plate"/>
+    <origin xyz="0.0 0.0 ${base_height}" rpy="0 0 0"/>
+    <axis xyz="0 0 1"/>
+    <limit velocity="4.8" effort="1" lower="${-pi*0.9}" upper="${pi*0.9}"/>
+    <!-- <limit velocity="4.8" effort="1" lower="${-pi/2}" upper="${pi/2}" /> -->
+  </joint>
+  <!--  Base_Plate -->
+  <link name="base_plate">
+    <visual>
+      <origin xyz="0 0 ${-base_plate_thickness/2}" rpy="0 0 0"/>
+      <geometry>
+        <cylinder radius="${base_plate_radii}" length="${base_plate_thickness}"/>
+      </geometry>
+      <material name="black"/>
+    </visual>
+    <collision>
+      <origin xyz="0 0 ${-base_plate_thickness/2}" rpy="0 0 0"/>
+      <geometry>
+        <cylinder radius="${base_plate_radii}" length="${base_plate_thickness}"/>
+      </geometry>
+    </collision>
+    <inertial>
+      <origin xyz="-3.0184870e-04 5.4043684e-04 ${0.018 + 2.9433464e-02}" />
+      <mass value="9.8406837e-02" />
+      <inertia ixx="3.4543422e-05" ixy="-1.6031095e-08" ixz="-3.8375155e-07"
+               iyy="3.2689329e-05" iyz="2.8511935e-08"
+               izz="1.8850320e-05" />
+    </inertial>
+  </link>
+  <!--  Base_Plate_Arm1_Joint -->
+  <joint name="base_plate_arm1_joint" type="revolute">
+    <parent link="base_plate"/>
+    <child link="arm1"/>
+    <origin xyz="0.0 0.0 0.060" rpy="0 0 0"/>
+    <axis xyz="0 1 0"/>
+    <limit velocity="4.8" effort="1" lower="${-pi * 0.9 / 2}" upper="${pi * 0.9 / 2}" />
+  </joint>
+  <xacro:Supp_Link parent="arm1" x="0" y="0" z="0.0" height="0.060"/>
+  <!--  Arm1 -->
+  <link name="arm1">
+    <visual>
+      <origin xyz="0 0 ${arm1_length/2}" rpy="0 0 0"/>
+      <geometry>
+        <box size="${arm1_width} ${arm1_width} ${arm1_length}"/>
+      </geometry>
+      <material name="black"/>
+    </visual>
+    <collision>
+      <origin xyz="0 0 ${arm1_length/2}" rpy="0 0 0"/>
+      <geometry>
+        <box size="${arm1_width} ${arm1_width} ${arm1_length}"/>
+      </geometry>
+    </collision>
+    <inertial>
+      <origin xyz="0 0 ${arm1_length/2}" />
+      <mass value="1.3850917e-01" />
+      <inertia ixx="3.3055381e-04" ixy="-9.7940978e-08" ixz="-3.8505711e-05"
+               iyy="3.4290447e-04" iyz="-1.5717516e-06"
+               izz="6.0346498e-05" />
+    </inertial>
+  </link>
+  <!--  Base_Plate_Arm2_Joint -->
+  <joint name="arm1_arm2_joint" type="revolute">
+    <parent link="arm1"/>
+    <child link="arm2"/>
+    <origin xyz="0.0 0.045 ${arm2_joint_height}" rpy="0 1.57 0"/>
+    <axis xyz="0 1 0"/>
+    <limit velocity="4.8" effort="1" lower="${-pi * 0.8 / 2}" upper="${pi * 0.8 / 2}" />
+  </joint>
+  <xacro:Supp_Link parent="arm2" x="0" y="-0.025" z="0" height="0.100"/>
+  <!--  Arm2 -->
+  <link name="arm2">
+    <visual>
+      <origin xyz="0 0 ${arm2_length/2}" rpy="0 0 0"/>
+      <geometry>
+        <box size="${arm2_width} ${arm2_width} ${arm2_length}"/>
+      </geometry>
+      <material name="black"/>
+    </visual>
+    <collision>
+      <origin xyz="0 0 ${arm2_length/2}" rpy="0 0 0"/>
+      <geometry>
+        <box size="${arm2_width} ${arm2_width} ${arm2_length}"/>
+      </geometry>
+    </collision>
+    <inertial>
+      <origin xyz="0 0 ${arm2_length/2}" />
+      <mass value="1.3274562e-01" />
+      <inertia ixx="3.0654178e-05" ixy="-1.2764155e-06" ixz="-2.6874417e-07"
+               iyy="2.4230292e-04" iyz="1.1559550e-08"
+               izz="2.5155057e-04" />
+    </inertial>
+  </link>
   <!--  EF_Holder_Joint -->
   <joint name="ef_holder_joint" type="fixed">
@@ -199,5 +213,5 @@
       <origin xyz="0 0 0" rpy="0 0 0"/>
       <geometry>
-        <mesh filename="package://proxygen_description/meshes/chain_link5.stl" scale="0.001 0.001 0.001"/>
+        <mesh filename="file://$(find proxygen_description)/meshes/chain_link5.stl" scale="0.001 0.001 0.001"/>
       </geometry>
       <material name="grey"/>
@@ -206,5 +220,5 @@
       <origin xyz="0 0 0" rpy="0 0 0"/>
       <geometry>
-        <mesh filename="package://proxygen_description/meshes/chain_link5.stl" scale="0.001 0.001 0.001"/>
+        <mesh filename="file://$(find proxygen_description)/meshes/chain_link5.stl" scale="0.001 0.001 0.001"/>
       </geometry>
     </collision>
@@ -222,5 +236,5 @@
       <origin xyz="0.0 0.0 0" rpy="0 0 0"/>
       <geometry>
-        <mesh filename="package://proxygen_description/meshes/chain_link_grip_l.stl" scale="0.001 0.001 0.001"/>
+        <mesh filename="file://$(find proxygen_description)/meshes/chain_link_grip_l.stl" scale="0.001 0.001 0.001"/>
       </geometry>
       <material name="grey"/>
@@ -229,5 +243,5 @@
       <origin xyz="0.0 0.0 0" rpy="0 0 0"/>
       <geometry>
-        <mesh filename="package://proxygen_description/meshes/chain_link_grip_l.stl" scale="0.001 0.001 0.001"/>
+        <mesh filename="file://$(find proxygen_description)/meshes/chain_link_grip_l.stl" scale="0.001 0.001 0.001"/>
       </geometry>
     </collision>
@@ -253,5 +267,5 @@
       <origin xyz="0.0 -0.0 0" rpy="0 0 0"/>
       <geometry>
-        <mesh filename="package://proxygen_description/meshes/chain_link_grip_r.stl" scale="0.001 0.001 0.001"/>
+        <mesh filename="file://$(find proxygen_description)/meshes/chain_link_grip_r.stl" scale="0.001 0.001 0.001"/>
       </geometry>
       <material name="grey"/>
@@ -260,5 +274,5 @@
       <origin xyz="0.0 -0.0 0" rpy="0 0 0"/>
       <geometry>
-        <mesh filename="package://proxygen_description/meshes/chain_link_grip_r.stl" scale="0.001 0.001 0.001"/>
+        <mesh filename="file://$(find proxygen_description)/meshes/chain_link_grip_r.stl" scale="0.001 0.001 0.001"/>
       </geometry>
     </collision>

File: proxygen_description/xacro/proxygen.xacro (robot description, xacro)
@@ -64,4 +64,20 @@
     </inertial>
   </link>
+  <!-- Dummy_Link -->
+  <link name="dummy_link">
+    <visual>
+      <origin xyz="0.0 0.0 ${base_height/2 + arm1_joint_height/2}" rpy="0 0 0"/>
+      <geometry>
+        <cylinder radius="0.030" length="${base_height + arm1_joint_height}"/>
+      </geometry>
+      <material name="grey"/>
+    </visual>
+  </link>
+  <!-- Dummy_Joint -->
+  <joint name="dummy_joint" type="fixed">
+    <parent link="base_link"/>
+    <child link="dummy_link"/>
+    <origin xyz="0 0 0" rpy="0 0 0"/>
+  </joint>
   <!-- Base_Link_Plate_Joint -->
   <joint name="base_link_plate_joint" type="revolute">
