Commit message: implemented ros2 controllers in gazebo ignition

File: proxygen_description/xacro/proxygen.main.xacro (robot description, xacro)
@@ -4,6 +4,7 @@
   <!-- Import Rviz colors -->
   <xacro:include filename="$(find proxygen_description)/xacro/materials.xacro" />
-  <!-- Import all Gazebo-customization elements, including Gazebo colors -->
-  <!-- <xacro:include filename="$(find proxygen_description)/xacro/proxygen.gazebo.xacro" /> -->
+  <!-- Import all ROS2-control elements -->
+  <!-- <xacro:include filename="$(find proxygen_description)/xacro/proxygen.gz.control.xacro" /> -->
+  <xacro:include filename="$(find proxygen_description)/xacro/proxygen.ign.control.xacro" />
   <!-- Import xacro -->
   <xacro:include filename="$(find proxygen_description)/xacro/proxygen.xacro" />

File: proxygen_description/xacro/proxygen.xacro (robot description, xacro)
@@ -1,4 +1,3 @@
 <?xml version="1.0"?>
-<!-- Open_Manipulator Chain -->
 <robot xmlns:xacro="http://ros.org/wiki/xacro">
 <xacro:property name="base_radii" value="0.100"/>
@@ -18,4 +17,13 @@
 <xacro:property name="arm1_length" value="${arm2_joint_height - arm1_width * 1.5 / 2}"/>
 <xacro:property name="arm2_length" value="${end_effector_joint_height}"/>
+<!-- Mass Properties -->
+<xacro:property name="supp_link_mass" value="1.5"/>
+<xacro:property name="base_link_mass" value="5.0"/>
+<xacro:property name="base_plate_mass" value="1.0"/>
+<xacro:property name="arm1_mass" value="0.5"/>
+<xacro:property name="arm2_mass" value="0.5"/>
+<xacro:property name="ef_holder_mass" value="0.1"/>
+<xacro:property name="gripper_mass" value="0.05"/>
+<xacro:property name="end_effector_mass" value="0.001"/>
   <xacro:macro name="Supp_Link" params="parent x y z height">
     <link name="supp_link${parent}">
@@ -29,8 +37,10 @@
       <inertial>
         <origin xyz="0 0 0" />
-        <mass value="9.8406837e-03" />
-        <inertia ixx="3.4543422e-06" ixy="-1.6031095e-07" ixz="-3.8375155e-08"
-                 iyy="3.2689329e-06"  iyz="2.8511935e-07"
-                 izz="1.8850320e-06" />
+        <mass value="${supp_link_mass}" />
+        <inertia ixx="${(supp_link_mass/12) * (3*0.04*0.04 + height*height)}"
+                 ixy="0" ixz="0"
+                 iyy="${(supp_link_mass/12) * (3*0.04*0.04 + height*height)}"
+                 iyz="0"
+                 izz="${(supp_link_mass * 0.04*0.04)/2}" />
       </inertial>
     </link>
@@ -57,9 +67,11 @@
     </collision>
     <inertial>
-      <origin xyz="3.0876154e-04 0.0000000e+00 -1.2176461e-04" />
-      <mass value="7.9119962e-02" />
-      <inertia ixx="1.2505234e-05" ixy="0.0" ixz="-1.7855208e-07"
-               iyy="2.1898364e-05" iyz="0.0"
-               izz="1.9267361e-05" />
+      <origin xyz="0 0 0" />
+      <mass value="${base_link_mass}" />
+      <inertia ixx="${(base_link_mass/12) * (3*base_radii*base_radii + base_height*base_height)}"
+               ixy="0" ixz="0"
+               iyy="${(base_link_mass/12) * (3*base_radii*base_radii + base_height*base_height)}"
+               iyz="0"
+               izz="${(base_link_mass * base_radii*base_radii)/2}" />
     </inertial>
   </link>
@@ -86,6 +98,5 @@
     <origin xyz="0.0 0.0 ${base_height}" rpy="0 0 0"/>
     <axis xyz="0 0 1"/>
-    <limit velocity="4.8" effort="1" lower="${-pi*0.9}" upper="${pi*0.9}"/>
-    <!-- <limit velocity="4.8" effort="1" lower="${-pi/2}" upper="${pi/2}" /> -->
+    <limit velocity="10" effort="20" lower="${-pi*0.9}" upper="${pi*0.9}"/>
   </joint>
   <!--  Base_Plate -->
@@ -105,9 +116,11 @@
     </collision>
     <inertial>
-      <origin xyz="-3.0184870e-04 5.4043684e-04 ${0.018 + 2.9433464e-02}" />
-      <mass value="9.8406837e-02" />
-      <inertia ixx="3.4543422e-05" ixy="-1.6031095e-08" ixz="-3.8375155e-07"
-               iyy="3.2689329e-05" iyz="2.8511935e-08"
-               izz="1.8850320e-05" />
+      <origin xyz="0 0 0" />
+      <mass value="${base_plate_mass}" />
+      <inertia ixx="${(base_plate_mass/12) * (3*base_plate_radii*base_plate_radii + base_plate_thickness*base_plate_thickness)}"
+               ixy="0" ixz="0"
+               iyy="${(base_plate_mass/12) * (3*base_plate_radii*base_plate_radii + base_plate_thickness*base_plate_thickness)}"
+               iyz="0"
+               izz="${(base_plate_mass * base_plate_radii*base_plate_radii)/2}" />
     </inertial>
   </link>
@@ -118,5 +131,5 @@
     <origin xyz="0.0 0.0 0.060" rpy="0 0 0"/>
     <axis xyz="0 1 0"/>
-    <limit velocity="4.8" effort="1" lower="${-pi * 0.9 / 2}" upper="${pi * 0.9 / 2}" />
+    <limit velocity="1000" effort="10000" lower="${-pi * 0.9 / 2}" upper="${pi * 0.9 / 2}" />
   </joint>
   <xacro:Supp_Link parent="arm1" x="0" y="0" z="0.0" height="0.060"/>
@@ -138,8 +151,10 @@
     <inertial>
       <origin xyz="0 0 ${arm1_length/2}" />
-      <mass value="1.3850917e-01" />
-      <inertia ixx="3.3055381e-04" ixy="-9.7940978e-08" ixz="-3.8505711e-05"
-               iyy="3.4290447e-04" iyz="-1.5717516e-06"
-               izz="6.0346498e-05" />
+      <mass value="${arm1_mass}" />
+      <inertia ixx="${(arm1_mass/12) * (arm1_width*arm1_width + arm1_length*arm1_length)}"
+               ixy="0" ixz="0"
+               iyy="${(arm1_mass/12) * (arm1_width*arm1_width + arm1_length*arm1_length)}"
+               iyz="0"
+               izz="${(arm1_mass/12) * (arm1_width*arm1_width + arm1_width*arm1_width)}" />
     </inertial>
   </link>
@@ -150,5 +165,5 @@
     <origin xyz="0.0 0.045 ${arm2_joint_height}" rpy="0 1.57 0"/>
     <axis xyz="0 1 0"/>
-    <limit velocity="4.8" effort="1" lower="${-pi * 0.8 / 2}" upper="${pi * 0.8 / 2}" />
+    <limit velocity="10" effort="20" lower="${-pi * 0.8 / 2}" upper="${pi * 0.8 / 2}" />
   </joint>
   <xacro:Supp_Link parent="arm2" x="0" y="-0.025" z="0" height="0.100"/>
@@ -170,8 +185,10 @@
     <inertial>
       <origin xyz="0 0 ${arm2_length/2}" />
-      <mass value="1.3274562e-01" />
-      <inertia ixx="3.0654178e-05" ixy="-1.2764155e-06" ixz="-2.6874417e-07"
-               iyy="2.4230292e-04" iyz="1.1559550e-08"
-               izz="2.5155057e-04" />
+      <mass value="${arm2_mass}" />
+      <inertia ixx="${(arm2_mass/12) * (arm2_width*arm2_width + arm2_length*arm2_length)}"
+               ixy="0" ixz="0"
+               iyy="${(arm2_mass/12) * (arm2_width*arm2_width + arm2_length*arm2_length)}"
+               iyz="0"
+               izz="${(arm2_mass/12) * (arm2_width*arm2_width + arm2_width*arm2_width)}" />
     </inertial>
   </link>
@@ -198,6 +215,6 @@
     </collision>
     <inertial>
-      <origin xyz="4.4206755e-02 3.6839985e-07 8.9142216e-03" />
-      <mass value="1.0e-03" />
+      <origin xyz="0 0 0" />
+      <mass value="${ef_holder_mass}" />
       <inertia ixx="1.0e-03" ixy="0.0" ixz="0.0"
                iyy="1.0e-03" iyz="0.0"
@@ -222,5 +239,5 @@
     <inertial>
       <origin xyz="0 0 0" />
-      <mass value="1.0e-03" />
+      <mass value="${gripper_mass}" />
       <inertia ixx="1.0e-03" ixy="0.0" ixz="0.0"
                iyy="1.0e-03" iyz="0.0"
@@ -234,5 +251,5 @@
     <origin xyz="0.0817 0.021 0.0" rpy="0 0 0"/>
     <axis xyz="0 1 0"/>
-    <limit velocity="4.8" effort="1" lower="-0.010" upper="0.019" />
+    <limit velocity="10" effort="20" lower="-0.010" upper="0.019" />
   </joint>
   <!--  Gripper link sub -->
@@ -253,5 +270,5 @@
     <inertial>
       <origin xyz="0 0 0" />
-      <mass value="1.0e-03" />
+      <mass value="${gripper_mass}" />
       <inertia ixx="1.0e-03" ixy="0.0" ixz="0.0"
                iyy="1.0e-03" iyz="0.0"
@@ -265,6 +282,6 @@
     <origin xyz="0.0817 -0.021 0" rpy="0 0 0"/>
     <axis xyz="0 -1 0"/>
-    <limit velocity="4.8" effort="1" lower="-0.010" upper="0.019" />
-    <mimic joint="gripper" multiplier="1"/>
+    <limit velocity="10" effort="20" lower="-0.010" upper="0.019" />
+    <!-- <mimic joint="gripper" multiplier="1"/> -->
   </joint>
   <!-- end effector joint -->
@@ -287,5 +304,5 @@
     <inertial>
       <origin xyz="0 0 0" />
-      <mass value="1.0e-03" />
+      <mass value="${end_effector_mass}" />
       <inertia ixx="1.0e-03" ixy="0.0" ixz="0.0"
                iyy="1.0e-03" iyz="0.0"
